File: PowerConversionBoard.sch (EAGLE design)
At the start: 48 parts, among them U1 LM2678, U2 LM2678

Commit message: ez fix
Connections:
- removed net N$20: C15.+, C16.+, C17.+, C18.+, C7.1, U1.VIN
- net +12V: now also C15.+, C16.+, C17.+, C18.+, C7.1, U1.VIN
Changed lines of the file:
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@@
 <pinref part="P+6" gate="1" pin="+12V"/>
 <wire x1="-18.542" y1="89.916" x2="-18.542" y2="62.738" width="0.1524" layer="91"/>
+<label x="-30.48" y="71.628" size="1.778" layer="95"/>
 </segment>
 <segment>
@@
 <label x="-37.4396" y="-210.6422" size="1.778" layer="95" xref="yes"/>
 <wire x1="-38.4556" y1="-210.6422" x2="-37.4396" y2="-210.6422" width="0.1524" layer="91"/>
+</segment>
+<segment>
+<pinref part="U1" gate="G$1" pin="VIN"/>
+<wire x1="17.018" y1="55.372" x2="19.812" y2="55.372" width="0.1524" layer="91"/>
+<wire x1="-49.022" y1="55.372" x2="-36.322" y2="55.372" width="0.1524" layer="91"/>
+<wire x1="-36.322" y1="55.372" x2="-23.622" y2="55.372" width="0.1524" layer="91"/>
+<wire x1="-23.622" y1="55.372" x2="-18.542" y2="55.372" width="0.1524" layer="91"/>
+<wire x1="-18.542" y1="55.372" x2="-10.922" y2="55.372" width="0.1524" layer="91"/>
+<wire x1="-10.922" y1="55.372" x2="1.778" y2="55.372" width="0.1524" layer="91"/>
+<wire x1="1.778" y1="45.212" x2="1.778" y2="55.372" width="0.1524" layer="91"/>
+<junction x="1.778" y="55.372"/>
+<pinref part="C15" gate="G$1" pin="+"/>
+<wire x1="-49.022" y1="45.212" x2="-49.022" y2="55.372" width="0.1524" layer="91"/>
+<pinref part="C16" gate="G$1" pin="+"/>
+<wire x1="-36.322" y1="45.212" x2="-36.322" y2="55.372" width="0.1524" layer="91"/>
+<junction x="-36.322" y="55.372"/>
+<pinref part="C17" gate="G$1" pin="+"/>
+<wire x1="-23.622" y1="45.212" x2="-23.622" y2="55.372" width="0.1524" layer="91"/>
+<junction x="-23.622" y="55.372"/>
+<pinref part="C18" gate="G$1" pin="+"/>
+<wire x1="-10.922" y1="45.212" x2="-10.922" y2="55.372" width="0.1524" layer="91"/>
+<junction x="-10.922" y="55.372"/>
+<pinref part="C7" gate="G$1" pin="1"/>
+<wire x1="-18.542" y1="63.5" x2="-18.542" y2="55.372" width="0.1524" layer="91"/>
+<junction x="-18.542" y="55.372"/>
+<wire x1="1.778" y1="55.372" x2="17.018" y2="55.372" width="0.1524" layer="91"/>
+<label x="-11.176" y="65.278" size="1.778" layer="95"/>
 </segment>
 </net>
@@
 </segment>
 </net>
-<net name="N$20" class="0">
-<segment>
-<pinref part="U1" gate="G$1" pin="VIN"/>
-<wire x1="17.018" y1="55.372" x2="19.812" y2="55.372" width="0.1524" layer="91"/>
-<wire x1="-49.022" y1="55.372" x2="-36.322" y2="55.372" width="0.1524" layer="91"/>
-<wire x1="-36.322" y1="55.372" x2="-23.622" y2="55.372" width="0.1524" layer="91"/>
-<wire x1="-23.622" y1="55.372" x2="-18.542" y2="55.372" width="0.1524" layer="91"/>
-<wire x1="-18.542" y1="55.372" x2="-10.922" y2="55.372" width="0.1524" layer="91"/>
-<wire x1="-10.922" y1="55.372" x2="1.778" y2="55.372" width="0.1524" layer="91"/>
-<wire x1="1.778" y1="45.212" x2="1.778" y2="55.372" width="0.1524" layer="91"/>
-<junction x="1.778" y="55.372"/>
-<pinref part="C15" gate="G$1" pin="+"/>
-<wire x1="-49.022" y1="45.212" x2="-49.022" y2="55.372" width="0.1524" layer="91"/>
-<pinref part="C16" gate="G$1" pin="+"/>
-<wire x1="-36.322" y1="45.212" x2="-36.322" y2="55.372" width="0.1524" layer="91"/>
-<junction x="-36.322" y="55.372"/>
-<pinref part="C17" gate="G$1" pin="+"/>
-<wire x1="-23.622" y1="45.212" x2="-23.622" y2="55.372" width="0.1524" layer="91"/>
-<junction x="-23.622" y="55.372"/>
-<pinref part="C18" gate="G$1" pin="+"/>
-<wire x1="-10.922" y1="45.212" x2="-10.922" y2="55.372" width="0.1524" layer="91"/>
-<junction x="-10.922" y="55.372"/>
-<pinref part="C7" gate="G$1" pin="1"/>
-<wire x1="-18.542" y1="63.5" x2="-18.542" y2="55.372" width="0.1524" layer="91"/>
-<junction x="-18.542" y="55.372"/>
-<wire x1="1.778" y1="55.372" x2="17.018" y2="55.372" width="0.1524" layer="91"/>
-</segment>
-</net>

Commit message: good progress
Connections:
- net +12V: now also U$12G$2.17, U$12G$2.18, U$12G$2.19, U$12G$2.20, U$12G$2.21, U$12G$2.22, U$12G$2.23, U$12G$2.24, U$12G$2.25, U$12G$2.26, U$12G$2.27, U$12G$2.28, U$12G$2.29, U$12G$2.30, U$12G$2.31, U$12G$2.32
- net +3.3V: now also U$12G$1.1, U$12G$1.10, U$12G$1.11, U$12G$1.12, U$12G$1.17, U$12G$1.18, U$12G$1.19, U$12G$1.2, U$12G$1.3, U$12G$1.4, U$12G$1.9
- net +5V: now also U$12G$1.13, U$12G$1.14, U$12G$1.15, U$12G$1.16, U$12G$1.22, U$12G$1.23, U$12G$1.24, U$12G$1.5, U$12G$1.6, U$12G$1.7, U$12G$1.8
- net CAN_H: now also U$12G$1.20
- net CAN_L: now also U$12G$1.21
- net GND: now also U$12G$2.1, U$12G$2.10, U$12G$2.11, U$12G$2.12, U$12G$2.13, U$12G$2.14, U$12G$2.15, U$12G$2.16, U$12G$2.2, U$12G$2.3, U$12G$2.4, U$12G$2.5, U$12G$2.6, U$12G$2.7, U$12G$2.8, U$12G$2.9
Changed lines of the file:
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@@
 <label x="-11.176" y="65.278" size="1.778" layer="95"/>
+</segment>
+<segment>
+<pinref part="U$12" gate="G$2" pin="17"/>
+<pinref part="U$12" gate="G$2" pin="20"/>
+<wire x1="124.46" y1="-233.68" x2="124.46" y2="-236.22" width="0.1524" layer="91"/>
+<pinref part="U$12" gate="G$2" pin="18"/>
+<wire x1="124.46" y1="-236.22" x2="124.46" y2="-238.76" width="0.1524" layer="91"/>
+<junction x="124.46" y="-236.22"/>
+<pinref part="U$12" gate="G$2" pin="19"/>
+<wire x1="124.46" y1="-238.76" x2="124.46" y2="-241.3" width="0.1524" layer="91"/>
+<junction x="124.46" y="-238.76"/>
+<label x="114.3" y="-243.586" size="1.778" layer="95"/>
+<pinref part="U$12" gate="G$2" pin="25"/>
+<pinref part="U$12" gate="G$2" pin="28"/>
+<wire x1="124.46" y1="-246.38" x2="124.46" y2="-248.92" width="0.1524" layer="91"/>
+<pinref part="U$12" gate="G$2" pin="26"/>
+<wire x1="124.46" y1="-248.92" x2="124.46" y2="-251.46" width="0.1524" layer="91"/>
+<junction x="124.46" y="-248.92"/>
+<pinref part="U$12" gate="G$2" pin="27"/>
+<wire x1="124.46" y1="-251.46" x2="124.46" y2="-254" width="0.1524" layer="91"/>
+<junction x="124.46" y="-251.46"/>
+<wire x1="124.46" y1="-241.3" x2="124.46" y2="-246.38" width="0.1524" layer="91"/>
+<junction x="124.46" y="-241.3"/>
+<junction x="124.46" y="-246.38"/>
+</segment>
+<segment>
+<pinref part="U$12" gate="G$2" pin="32"/>
+<pinref part="U$12" gate="G$2" pin="21"/>
+<wire x1="147.32" y1="-254" x2="147.32" y2="-251.46" width="0.1524" layer="91"/>
+<pinref part="U$12" gate="G$2" pin="22"/>
+<wire x1="147.32" y1="-251.46" x2="147.32" y2="-248.92" width="0.1524" layer="91"/>
+<wire x1="147.32" y1="-248.92" x2="147.32" y2="-246.38" width="0.1524" layer="91"/>
+<wire x1="147.32" y1="-246.38" x2="147.32" y2="-241.3" width="0.1524" layer="91"/>
+<wire x1="147.32" y1="-241.3" x2="147.32" y2="-238.76" width="0.1524" layer="91"/>
+<wire x1="147.32" y1="-238.76" x2="147.32" y2="-236.22" width="0.1524" layer="91"/>
+<wire x1="147.32" y1="-236.22" x2="147.32" y2="-233.68" width="0.1524" layer="91"/>
+<junction x="147.32" y="-236.22"/>
+<pinref part="U$12" gate="G$2" pin="23"/>
+<junction x="147.32" y="-238.76"/>
+<pinref part="U$12" gate="G$2" pin="24"/>
+<junction x="147.32" y="-241.3"/>
+<pinref part="U$12" gate="G$2" pin="29"/>
+<junction x="147.32" y="-246.38"/>
+<pinref part="U$12" gate="G$2" pin="30"/>
+<junction x="147.32" y="-248.92"/>
+<pinref part="U$12" gate="G$2" pin="31"/>
+<junction x="147.32" y="-251.46"/>
+<label x="155.702" y="-243.332" size="1.778" layer="95"/>
 </segment>
 </net>
@@
 <wire x1="-18.1356" y1="-215.7222" x2="-19.1516" y2="-215.7222" width="0.1524" layer="91"/>
 </segment>
+<segment>
+<pinref part="U$12" gate="G$2" pin="1"/>
+<pinref part="U$12" gate="G$2" pin="12"/>
+<wire x1="124.46" y1="-205.74" x2="124.46" y2="-208.28" width="0.1524" layer="91"/>
+<pinref part="U$12" gate="G$2" pin="2"/>
+<wire x1="124.46" y1="-208.28" x2="124.46" y2="-210.82" width="0.1524" layer="91"/>
+<junction x="124.46" y="-208.28"/>
+<pinref part="U$12" gate="G$2" pin="3"/>
+<wire x1="124.46" y1="-210.82" x2="124.46" y2="-213.36" width="0.1524" layer="91"/>
+<junction x="124.46" y="-210.82"/>
+<pinref part="U$12" gate="G$2" pin="4"/>
+<wire x1="124.46" y1="-213.36" x2="124.46" y2="-218.44" width="0.1524" layer="91"/>
+<junction x="124.46" y="-213.36"/>
+<pinref part="U$12" gate="G$2" pin="9"/>
+<wire x1="124.46" y1="-218.44" x2="124.46" y2="-220.98" width="0.1524" layer="91"/>
+<junction x="124.46" y="-218.44"/>
+<pinref part="U$12" gate="G$2" pin="10"/>
+<wire x1="124.46" y1="-220.98" x2="124.46" y2="-223.52" width="0.1524" layer="91"/>
+<junction x="124.46" y="-220.98"/>
+<pinref part="U$12" gate="G$2" pin="11"/>
+<wire x1="124.46" y1="-223.52" x2="124.46" y2="-226.06" width="0.1524" layer="91"/>
+<junction x="124.46" y="-223.52"/>
+<label x="115.824" y="-216.408" size="1.778" layer="95"/>
+</segment>
+<segment>
+<pinref part="U$12" gate="G$2" pin="5"/>
+<pinref part="U$12" gate="G$2" pin="16"/>
+<wire x1="147.32" y1="-205.74" x2="147.32" y2="-208.28" width="0.1524" layer="91"/>
+<pinref part="U$12" gate="G$2" pin="6"/>
+<wire x1="147.32" y1="-208.28" x2="147.32" y2="-210.82" width="0.1524" layer="91"/>
+<junction x="147.32" y="-208.28"/>
+<pinref part="U$12" gate="G$2" pin="7"/>
+<wire x1="147.32" y1="-210.82" x2="147.32" y2="-213.36" width="0.1524" layer="91"/>
+<junction x="147.32" y="-210.82"/>
+<pinref part="U$12" gate="G$2" pin="8"/>
+<wire x1="147.32" y1="-213.36" x2="147.32" y2="-218.44" width="0.1524" layer="91"/>
+<junction x="147.32" y="-213.36"/>
+<pinref part="U$12" gate="G$2" pin="13"/>
+<wire x1="147.32" y1="-218.44" x2="147.32" y2="-220.98" width="0.1524" layer="91"/>
+<junction x="147.32" y="-218.44"/>
+<pinref part="U$12" gate="G$2" pin="14"/>
+<wire x1="147.32" y1="-220.98" x2="147.32" y2="-223.52" width="0.1524" layer="91"/>
+<junction x="147.32" y="-220.98"/>
+<pinref part="U$12" gate="G$2" pin="15"/>
+<wire x1="147.32" y1="-223.52" x2="147.32" y2="-226.06" width="0.1524" layer="91"/>
+<junction x="147.32" y="-223.52"/>
+<label x="152.4" y="-215.646" size="1.778" layer="95"/>
+</segment>
 </net>
 <net name="+5V" class="0">
@@
 <pinref part="U$11" gate="G$1" pin="P$1"/>
 </segment>
+<segment>
+<pinref part="U$12" gate="G$1" pin="8"/>
+<pinref part="U$12" gate="G$1" pin="5"/>
+<wire x1="193.04" y1="-218.44" x2="193.04" y2="-215.9" width="0.1524" layer="91"/>
+<pinref part="U$12" gate="G$1" pin="6"/>
+<wire x1="193.04" y1="-215.9" x2="193.04" y2="-213.36" width="0.1524" layer="91"/>
+<wire x1="193.04" y1="-213.36" x2="193.04" y2="-210.82" width="0.1524" layer="91"/>
+<junction x="193.04" y="-213.36"/>
+<pinref part="U$12" gate="G$1" pin="7"/>
+<junction x="193.04" y="-215.9"/>
+<label x="186.944" y="-215.138" size="1.778" layer="95"/>
+</segment>
+<segment>
+<pinref part="U$12" gate="G$1" pin="16"/>
+<pinref part="U$12" gate="G$1" pin="13"/>
+<wire x1="193.04" y1="-238.76" x2="193.04" y2="-236.22" width="0.1524" layer="91"/>
+<pinref part="U$12" gate="G$1" pin="14"/>
+<wire x1="193.04" y1="-236.22" x2="193.04" y2="-233.68" width="0.1524" layer="91"/>
+<wire x1="193.04" y1="-233.68" x2="193.04" y2="-231.14" width="0.1524" layer="91"/>
+<junction x="193.04" y="-233.68"/>
+<pinref part="U$12" gate="G$1" pin="15"/>
+<junction x="193.04" y="-236.22"/>
+<label x="186.69" y="-235.458" size="1.778" layer="95"/>
+</segment>
+<segment>
+<pinref part="U$12" gate="G$1" pin="24"/>
+<pinref part="U$12" gate="G$1" pin="22"/>
+<wire x1="193.04" y1="-259.08" x2="193.04" y2="-256.54" width="0.1524" layer="91"/>
+<pinref part="U$12" gate="G$1" pin="23"/>
+<wire x1="193.04" y1="-256.54" x2="193.04" y2="-254" width="0.1524" layer="91"/>
+<junction x="193.04" y="-256.54"/>
+<label x="187.198" y="-256.54" size="1.778" layer="95"/>
+</segment>
 </net>
 <net name="+3.3V" class="0">
@@
 <label x="-19.1516" y="-205.5622" size="1.778" layer="95" rot="R180" xref="yes"/>
 <wire x1="-18.1356" y1="-205.5622" x2="-19.1516" y2="-205.5622" width="0.1524" layer="91"/>
+</segment>
+<segment>
+<pinref part="U$12" gate="G$1" pin="1"/>
+<pinref part="U$12" gate="G$1" pin="4"/>
+<wire x1="193.04" y1="-200.66" x2="193.04" y2="-203.2" width="0.1524" layer="91"/>
+<pinref part="U$12" gate="G$1" pin="2"/>
+<wire x1="193.04" y1="-203.2" x2="193.04" y2="-205.74" width="0.1524" layer="91"/>
+<junction x="193.04" y="-203.2"/>
+<pinref part="U$12" gate="G$1" pin="3"/>
+<wire x1="193.04" y1="-205.74" x2="193.04" y2="-208.28" width="0.1524" layer="91"/>
+<junction x="193.04" y="-205.74"/>
+<label x="185.674" y="-205.232" size="1.778" layer="95"/>
+</segment>
+<segment>
+<pinref part="U$12" gate="G$1" pin="9"/>
+<pinref part="U$12" gate="G$1" pin="12"/>
+<wire x1="193.04" y1="-220.98" x2="193.04" y2="-223.52" width="0.1524" layer="91"/>
+<pinref part="U$12" gate="G$1" pin="10"/>
+<wire x1="193.04" y1="-223.52" x2="193.04" y2="-226.06" width="0.1524" layer="91"/>
+<junction x="193.04" y="-223.52"/>
+<pinref part="U$12" gate="G$1" pin="11"/>
+<wire x1="193.04" y1="-226.06" x2="193.04" y2="-228.6" width="0.1524" layer="91"/>
+<junction x="193.04" y="-226.06"/>
+<label x="185.42" y="-225.044" size="1.778" layer="95"/>
+</segment>
+<segment>
+<pinref part="U$12" gate="G$1" pin="17"/>
+<pinref part="U$12" gate="G$1" pin="19"/>
+<wire x1="193.04" y1="-241.3" x2="193.04" y2="-243.84" width="0.1524" layer="91"/>
+<pinref part="U$12" gate="G$1" pin="18"/>
+<wire x1="193.04" y1="-243.84" x2="193.04" y2="-246.38" width="0.1524" layer="91"/>
+<junction x="193.04" y="-243.84"/>
+<label x="184.404" y="-243.586" size="1.778" layer="95"/>
 </segment>
 </net>
@@
 <pinref part="U$9" gate="G$1" pin="47"/>
 </segment>
+<segment>
+<pinref part="U$12" gate="G$1" pin="20"/>
+<wire x1="193.04" y1="-248.92" x2="189.23" y2="-248.92" width="0.1524" layer="91"/>
+<label x="178.816" y="-248.666" size="1.778" layer="95"/>
+</segment>
 </net>
 <net name="CAN_L" class="0">
@@
 <pinref part="U$9" gate="G$1" pin="48"/>
 </segment>
-</net>
+<segment>
+<pinref part="U$12" gate="G$1" pin="21"/>
+<wire x1="193.04" y1="-251.46" x2="189.23" y2="-251.46" width="0.1524" layer="91"/>
+<label x="179.578" y="-251.714" size="1.778" layer="95"/>
+</segment>
+</net>

Commit message: k
Parts:
- renumbered J1 to 12V, J2 to GND, J3 to GND3, J5 to +3.3V, J6 to +5V, U$10 to GND2, U$11 to 5V, U$5 to +12V, U$6 to +3.3
Changed lines of the file:
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@@
 <part name="C7" library="rcl" library_urn="urn:adsk.eagle:library:334" deviceset="C-EU" device="C0603" package3d_urn="urn:adsk.eagle:package:23616/2" value="0.47uF"/>
 <part name="P+6" library="supply1" library_urn="urn:adsk.eagle:library:371" deviceset="+12V" device=""/>
-<part name="J1" library="SparkFun-Connectors" library_urn="urn:adsk.eagle:library:513" deviceset="BANANA_CONN" device="" package3d_urn="urn:adsk.eagle:package:38018/1"/>
-<part name="J2" library="SparkFun-Connectors" library_urn="urn:adsk.eagle:library:513" deviceset="BANANA_CONN" device="" package3d_urn="urn:adsk.eagle:package:38018/1"/>
+<part name="12V" library="SparkFun-Connectors" library_urn="urn:adsk.eagle:library:513" deviceset="BANANA_CONN" device="" package3d_urn="urn:adsk.eagle:package:38018/1"/>
+<part name="GND" library="SparkFun-Connectors" library_urn="urn:adsk.eagle:library:513" deviceset="BANANA_CONN" device="" package3d_urn="urn:adsk.eagle:package:38018/1"/>
 <part name="P+5" library="supply1" library_urn="urn:adsk.eagle:library:371" deviceset="+12V" device=""/>
-<part name="J6" library="SparkFun-Connectors" library_urn="urn:adsk.eagle:library:513" deviceset="BANANA_CONN" device="" package3d_urn="urn:adsk.eagle:package:38018/1"/>
+<part name="+5V" library="SparkFun-Connectors" library_urn="urn:adsk.eagle:library:513" deviceset="BANANA_CONN" device="" package3d_urn="urn:adsk.eagle:package:38018/1"/>
 <part name="P+2" library="supply1" library_urn="urn:adsk.eagle:library:371" deviceset="+12V" device=""/>
-<part name="J5" library="SparkFun-Connectors" library_urn="urn:adsk.eagle:library:513" deviceset="BANANA_CONN" device="" package3d_urn="urn:adsk.eagle:package:38018/1"/>
-<part name="J3" library="SparkFun-Connectors" library_urn="urn:adsk.eagle:library:513" deviceset="BANANA_CONN" device="" package3d_urn="urn:adsk.eagle:package:38018/1"/>
+<part name="+3.3V" library="SparkFun-Connectors" library_urn="urn:adsk.eagle:library:513" deviceset="BANANA_CONN" device="" package3d_urn="urn:adsk.eagle:package:38018/1"/>
+<part name="GND3" library="SparkFun-Connectors" library_urn="urn:adsk.eagle:library:513" deviceset="BANANA_CONN" device="" package3d_urn="urn:adsk.eagle:package:38018/1"/>
 <part name="J4" library="SparkFun-Connectors" library_urn="urn:adsk.eagle:library:513" deviceset="BANANA_CONN" device="" package3d_urn="urn:adsk.eagle:package:38018/1"/>
 <part name="D1" library="SparkFun-LED" library_urn="urn:adsk.eagle:library:529" deviceset="LED" device="0603" package3d_urn="urn:adsk.eagle:package:39354/1"/>
@@
 <part name="U$7" library="HCM1305" deviceset="HCM1305" device=""/>
 <part name="U$2" library="HCM1305" deviceset="HCM1305" device=""/>
-<part name="U$5" library="TP" deviceset="TP" device=""/>
-<part name="U$10" library="TP" deviceset="TP" device=""/>
-<part name="U$11" library="TP" deviceset="TP" device=""/>
-<part name="U$6" library="TP" deviceset="TP" device=""/>
+<part name="+12V" library="TP" deviceset="TP" device=""/>
+<part name="GND2" library="TP" deviceset="TP" device=""/>
+<part name="5V" library="TP" deviceset="TP" device=""/>
+<part name="+3.3" library="TP" deviceset="TP" device=""/>
 <part name="U$8" library="TP" deviceset="TP" device=""/>
 <part name="U$12" library="ET60S-02-24-02-X-VP-GP" deviceset="ET60S-02-24-02-X-VP-GP" device=""/>
@@
 <attribute name="VALUE" x="-21.082" y="87.376" size="1.778" layer="96" rot="R90"/>
 </instance>
-<instance part="J1" gate="G$1" x="-98.298" y="11.43" smashed="yes">
+<instance part="12V" gate="G$1" x="-98.298" y="11.43" smashed="yes">
 <attribute name="NAME" x="-99.314" y="13.208" size="1.778" layer="95" font="vector"/>
 <attribute name="VALUE" x="-99.314" y="8.382" size="1.778" layer="96" font="vector"/>
 </instance>
-<instance part="J2" gate="G$1" x="-98.298" y="3.81" smashed="yes">
+<instance part="GND" gate="G$1" x="-98.298" y="3.81" smashed="yes">
 <attribute name="NAME" x="-99.314" y="5.588" size="1.778" layer="95" font="vector"/>
 <attribute name="VALUE" x="-99.314" y="0.762" size="1.778" layer="96" font="vector"/>
@@
 <attribute name="VALUE" x="-103.378" y="8.89" size="1.778" layer="96" rot="R180"/>
 </instance>
-<instance part="J6" gate="G$1" x="-98.298" y="-4.064" smashed="yes">
+<instance part="+5V" gate="G$1" x="-98.298" y="-4.064" smashed="yes">
 <attribute name="NAME" x="-99.314" y="-2.286" size="1.778" layer="95" font="vector"/>
 <attribute name="VALUE" x="-99.314" y="-7.112" size="1.778" layer="96" font="vector"/>
@@
 <attribute name="VALUE" x="-76.708" y="11.938" size="1.778" layer="96" rot="R180"/>
 </instance>
-<instance part="J5" gate="G$1" x="443.484" y="-5.334" smashed="yes">
+<instance part="+3.3V" gate="G$1" x="443.484" y="-5.334" smashed="yes">
 <attribute name="NAME" x="442.468" y="-3.556" size="1.778" layer="95" font="vector"/>
 <attribute name="VALUE" x="442.468" y="-8.382" size="1.778" layer="96" font="vector"/>
 </instance>
-<instance part="J3" gate="G$1" x="443.23" y="-13.208" smashed="yes">
+<instance part="GND3" gate="G$1" x="443.23" y="-13.208" smashed="yes">
 <attribute name="NAME" x="442.214" y="-11.43" size="1.778" layer="95" font="vector"/>
 <attribute name="VALUE" x="442.214" y="-16.256" size="1.778" layer="96" font="vector"/>
@@
 <attribute name="NAME" x="85.83638125" y="57.919809375" size="1.78346875" layer="95"/>
 </instance>
-<instance part="U$5" gate="G$1" x="-71.628" y="14.478" smashed="yes" rot="R270">
+<instance part="+12V" gate="G$1" x="-71.628" y="14.478" smashed="yes" rot="R270">
 <attribute name="NAME" x="-69.088" y="12.7" size="1.778" layer="95" rot="R270"/>
 </instance>
-<instance part="U$10" gate="G$1" x="-71.628" y="4.826" smashed="yes" rot="R270">
+<instance part="GND2" gate="G$1" x="-71.628" y="4.826" smashed="yes" rot="R270">
 <attribute name="NAME" x="-69.088" y="3.048" size="1.778" layer="95" rot="R270"/>
 </instance>
-<instance part="U$11" gate="G$1" x="-71.628" y="-5.08" smashed="yes" rot="R270">
+<instance part="5V" gate="G$1" x="-71.628" y="-5.08" smashed="yes" rot="R270">
 <attribute name="NAME" x="-69.088" y="-6.858" size="1.778" layer="95" rot="R270"/>
 </instance>
-<instance part="U$6" gate="G$1" x="477.266" y="-5.588" smashed="yes" rot="R270">
+<instance part="+3.3" gate="G$1" x="477.266" y="-5.588" smashed="yes" rot="R270">
 <attribute name="NAME" x="479.806" y="-7.366" size="1.778" layer="95" rot="R270"/>
 </instance>
@@
 </segment>
 <segment>
-<pinref part="J1" gate="G$1" pin="1"/>
+<pinref part="12V" gate="G$1" pin="1"/>
 <pinref part="P+5" gate="1" pin="+12V"/>
 <wire x1="-100.838" y1="11.43" x2="-105.918" y2="11.43" width="0.1524" layer="91"/>
@@
 <pinref part="P+2" gate="1" pin="+12V"/>
 <wire x1="-74.168" y1="14.478" x2="-79.248" y2="14.478" width="0.1524" layer="91"/>
-<pinref part="U$5" gate="G$1" pin="P$1"/>
+<pinref part="+12V" gate="G$1" pin="P$1"/>
 </segment>
 <segment>
@@
 </segment>
 <segment>
-<pinref part="J2" gate="G$1" pin="1"/>
+<pinref part="GND" gate="G$1" pin="1"/>
 <wire x1="-100.838" y1="3.81" x2="-108.458" y2="3.81" width="0.1524" layer="91"/>
 <label x="-108.458" y="3.81" size="1.778" layer="95" rot="R180" xref="yes"/>
@@
 <wire x1="-74.168" y1="4.826" x2="-81.788" y2="4.826" width="0.1524" layer="91"/>
 <label x="-81.788" y="4.826" size="1.778" layer="95" rot="R180" xref="yes"/>
-<pinref part="U$10" gate="G$1" pin="P$1"/>
-</segment>
-<segment>
-<pinref part="J3" gate="G$1" pin="1"/>
+<pinref part="GND2" gate="G$1" pin="P$1"/>
+</segment>
+<segment>
+<pinref part="GND3" gate="G$1" pin="1"/>
 <wire x1="440.69" y1="-13.208" x2="433.07" y2="-13.208" width="0.1524" layer="91"/>
 <label x="433.07" y="-13.208" size="1.778" layer="95" rot="R180" xref="yes"/>
@@
 </segment>
 <segment>
-<pinref part="J6" gate="G$1" pin="1"/>
+<pinref part="+5V" gate="G$1" pin="1"/>
 <wire x1="-100.838" y1="-4.064" x2="-108.458" y2="-4.064" width="0.1524" layer="91"/>
 <label x="-108.458" y="-4.064" size="1.778" layer="95" rot="R180" xref="yes"/>
@@
 <wire x1="-74.168" y1="-5.08" x2="-81.788" y2="-5.08" width="0.1524" layer="91"/>
 <label x="-81.788" y="-5.08" size="1.778" layer="95" rot="R180" xref="yes"/>
-<pinref part="U$11" gate="G$1" pin="P$1"/>
+<pinref part="5V" gate="G$1" pin="P$1"/>
 </segment>
 <segment>
@@
 </segment>
 <segment>
-<pinref part="J5" gate="G$1" pin="1"/>
+<pinref part="+3.3V" gate="G$1" pin="1"/>
 <wire x1="440.944" y1="-5.334" x2="433.324" y2="-5.334" width="0.1524" layer="91"/>
 <label x="433.324" y="-5.334" size="1.778" layer="95" rot="R180" xref="yes"/>
@@
 <wire x1="474.726" y1="-5.588" x2="467.106" y2="-5.588" width="0.1524" layer="91"/>
 <label x="467.106" y="-5.588" size="1.778" layer="95" rot="R180" xref="yes"/>
-<pinref part="U$6" gate="G$1" pin="P$1"/>
-</segment>
-<segment>
+<pinref part="+3.3" gate="G$1" pin="P$1"/>
+</segment>
+<segment>
